Commit message: Add urdf/srdf/mesh files for RG6-v2 gripper

File: onrobot_description/urdf/onrobot_rg.srdf.xacro (robot description, xacro)
@@ -28,4 +28,7 @@
     <xacro:macro name="onrobot_rg2_group" params="prefix">
         <xacro:onrobot_rg_group model="rg2_v1" prefix="${prefix}"/>
+    </xacro:macro>
+    <xacro:macro name="onrobot_rg6_v2_group" params="prefix">
+        <xacro:onrobot_rg_group model="rg6_v2" prefix="${prefix}"/>
     </xacro:macro>
     <xacro:macro name="onrobot_rg_autocol" params="model prefix">
@@ -157,4 +160,7 @@
         <xacro:onrobot_rg_autocol model="rg6_v1" prefix="${prefix}"/>
     </xacro:macro>
+    <xacro:macro name="onrobot_rg6_v2_autocol" params="prefix">
+        <xacro:onrobot_rg_autocol model="rg6_v2" prefix="${prefix}"/>
+    </xacro:macro>
     <xacro:macro name="onrobot_rg_col_with" params="model prefix link">
         <xacro:if value="${model == 'rg6_v1'}">
@@ -179,3 +185,6 @@
         <xacro:onrobot_rg_col_with model="rg6_v1" prefix="${prefix}" link="${link}"/>
     </xacro:macro>
+    <xacro:macro name="onrobot_rg6_v2_col_with" params="prefix link">
+        <xacro:onrobot_rg_col_with model="rg6_v2" prefix="${prefix}" link="${link}"/>
+    </xacro:macro>
 </robot>

Commit message: Fix rg6-v2 srdf for safety_shields

File: onrobot_description/urdf/onrobot_rg.srdf.xacro (robot description, xacro)
@@ -7,4 +7,8 @@
     <xacro:macro name="onrobot_rg_group" params="model prefix">
         <xacro:if value="${model == 'rg6_v1'}">
+            <link name="${prefix}_finger_1_safety_shield"/>
+            <link name="${prefix}_finger_2_safety_shield"/>
+        </xacro:if>
+        <xacro:if value="${model == 'rg6_v2'}">
             <link name="${prefix}_finger_1_safety_shield"/>
             <link name="${prefix}_finger_2_safety_shield"/>
@@ -34,4 +38,24 @@
     <xacro:macro name="onrobot_rg_autocol" params="model prefix">
         <xacro:if value="${model == 'rg6_v1'}">
+            <disable_collisions link1="${prefix}_finger_1_safety_shield" link2="${prefix}_bracket" reason="Never"/>
+            <disable_collisions link1="${prefix}_finger_1_safety_shield" link2="${prefix}_finger_1_moment_arm" reason="Never"/>
+            <disable_collisions link1="${prefix}_finger_1_safety_shield" link2="${prefix}_finger_1_finger_tip" reason="Never"/>
+            <disable_collisions link1="${prefix}_finger_1_safety_shield" link2="${prefix}_finger_1_flex_finger" reason="Never"/>
+            <disable_collisions link1="${prefix}_finger_1_safety_shield" link2="${prefix}_finger_1_truss_arm" reason="Never"/>
+            <disable_collisions link1="${prefix}_finger_1_safety_shield" link2="${prefix}_finger_2_moment_arm" reason="Never"/>
+            <disable_collisions link1="${prefix}_finger_1_safety_shield" link2="${prefix}_finger_2_finger_tip" reason="Never"/>
+            <disable_collisions link1="${prefix}_finger_1_safety_shield" link2="${prefix}_finger_2_flex_finger" reason="Never"/>
+            <disable_collisions link1="${prefix}_finger_1_safety_shield" link2="${prefix}_finger_2_truss_arm" reason="Never"/>
+            <disable_collisions link1="${prefix}_finger_2_safety_shield" link2="${prefix}_bracket" reason="Never"/>
+            <disable_collisions link1="${prefix}_finger_2_safety_shield" link2="${prefix}_finger_1_moment_arm" reason="Never"/>
+            <disable_collisions link1="${prefix}_finger_2_safety_shield" link2="${prefix}_finger_1_finger_tip" reason="Never"/>
+            <disable_collisions link1="${prefix}_finger_2_safety_shield" link2="${prefix}_finger_1_flex_finger" reason="Never"/>
+            <disable_collisions link1="${prefix}_finger_2_safety_shield" link2="${prefix}_finger_1_truss_arm" reason="Never"/>
+            <disable_collisions link1="${prefix}_finger_2_safety_shield" link2="${prefix}_finger_2_moment_arm" reason="Never"/>
+            <disable_collisions link1="${prefix}_finger_2_safety_shield" link2="${prefix}_finger_2_finger_tip" reason="Never"/>
+            <disable_collisions link1="${prefix}_finger_2_safety_shield" link2="${prefix}_finger_2_flex_finger" reason="Never"/>
+            <disable_collisions link1="${prefix}_finger_2_safety_shield" link2="${prefix}_finger_2_truss_arm" reason="Never"/>
+        </xacro:if>
+        <xacro:if value="${model == 'rg6_v2'}">
             <disable_collisions link1="${prefix}_finger_1_safety_shield" link2="${prefix}_bracket" reason="Never"/>
             <disable_collisions link1="${prefix}_finger_1_safety_shield" link2="${prefix}_finger_1_moment_arm" reason="Never"/>
@@ -168,4 +192,8 @@
             <disable_collisions link1="${prefix}_finger_2_safety_shield" link2="${link}" reason="Never"/>
         </xacro:if>
+        <xacro:if value="${model == 'rg6_v2'}">
+            <disable_collisions link1="${prefix}_finger_1_safety_shield" link2="${link}" reason="Never"/>
+            <disable_collisions link1="${prefix}_finger_2_safety_shield" link2="${link}" reason="Never"/>
+        </xacro:if>
         <disable_collisions link1="${prefix}_bracket" link2="${link}" reason="Never"/>
         <disable_collisions link1="${prefix}_finger_1_moment_arm" link2="${link}" reason="Never"/>

Commit message: Follow new xacro srdf standard

File: onrobot_description/urdf/onrobot_rg.srdf.xacro (robot description, xacro)
@@ -5,34 +5,44 @@
 -->
 <robot xmlns:xacro="http://wiki.ros.org/xacro">
-    <xacro:macro name="onrobot_rg_group" params="model prefix">
-        <xacro:if value="${model == 'rg6_v1'}">
-            <link name="${prefix}_finger_1_safety_shield"/>
-            <link name="${prefix}_finger_2_safety_shield"/>
-        </xacro:if>
-        <xacro:if value="${model == 'rg6_v2'}">
-            <link name="${prefix}_finger_1_safety_shield"/>
-            <link name="${prefix}_finger_2_safety_shield"/>
-        </xacro:if>
-        <link name="${prefix}_bracket"/>
-        <link name="${prefix}_body"/>
-        <link name="${prefix}_finger_1_moment_arm"/>
-        <link name="${prefix}_finger_1_finger_tip"/>
-        <link name="${prefix}_finger_1_flex_finger"/>
-        <link name="${prefix}_finger_1_truss_arm"/>
-        <link name="${prefix}_finger_2_moment_arm"/>
-        <link name="${prefix}_finger_2_finger_tip"/>
-        <link name="${prefix}_finger_2_flex_finger"/>
-        <link name="${prefix}_finger_2_truss_arm"/>
-        <joint name="${prefix}_joint"/>
-        <passive_joint name="${prefix}_mirror_joint"/>
-    </xacro:macro>
-    <xacro:macro name="onrobot_rg6_group" params="prefix">
-        <xacro:onrobot_rg_group model="rg6_v1" prefix="${prefix}"/>
-    </xacro:macro>
-    <xacro:macro name="onrobot_rg2_group" params="prefix">
-        <xacro:onrobot_rg_group model="rg2_v1" prefix="${prefix}"/>
-    </xacro:macro>
-    <xacro:macro name="onrobot_rg6_v2_group" params="prefix">
-        <xacro:onrobot_rg_group model="rg6_v2" prefix="${prefix}"/>
+    <xacro:macro name="onrobot_rg_group_define" params="model group_name prefix">
+        <group name="${group_name}">
+            <xacro:if value="${model == 'rg6_v1'}">
+                <link name="${prefix}_finger_1_safety_shield"/>
+                <link name="${prefix}_finger_2_safety_shield"/>
+            </xacro:if>
+            <xacro:if value="${model == 'rg6_v2'}">
+                <link name="${prefix}_finger_1_safety_shield"/>
+                <link name="${prefix}_finger_2_safety_shield"/>
+            </xacro:if>
+            <link name="${prefix}_bracket"/>
+            <link name="${prefix}_body"/>
+            <link name="${prefix}_finger_1_moment_arm"/>
+            <link name="${prefix}_finger_1_finger_tip"/>
+            <link name="${prefix}_finger_1_flex_finger"/>
+            <link name="${prefix}_finger_1_truss_arm"/>
+            <link name="${prefix}_finger_2_moment_arm"/>
+            <link name="${prefix}_finger_2_finger_tip"/>
+            <link name="${prefix}_finger_2_flex_finger"/>
+            <link name="${prefix}_finger_2_truss_arm"/>
+            <joint name="${prefix}_joint"/>
+            <passive_joint name="${prefix}_mirror_joint"/>
+        </group>
+        <group_state name="open" group="${group_name}">
+            <joint name="${group_name}_joint" value="0.0"/>
+            <joint name="${group_name}_mirror_joint" value="0.0"/>
+        </group_state>
+        <group_state name="close" group="${group_name}">
+            <joint name="${group_name}_joint" value="1.3"/>
+            <joint name="${group_name}_mirror_joint" value="1.3"/>
+        </group_state>
+    </xacro:macro>
+    <xacro:macro name="onrobot_rg6_group_define" params="group_name prefix">
+        <xacro:onrobot_rg_group_define model="rg6_v1" group_name="${group_name}" prefix="${prefix}"/>
+    </xacro:macro>
+    <xacro:macro name="onrobot_rg2_group_define" params="group_name prefix">
+        <xacro:onrobot_rg_group_define model="rg2_v1" group_name="${group_name}" prefix="${prefix}"/>
+    </xacro:macro>
+    <xacro:macro name="onrobot_rg6_v2_group_define" params="group_name prefix">
+        <xacro:onrobot_rg_group_define model="rg6_v2" group_name="${group_name}" prefix="${prefix}"/>
     </xacro:macro>
     <xacro:macro name="onrobot_rg_autocol" params="model prefix">
