Commit message: Create "standard" srdf using xacro + minor fixes

File: onrobot_description/urdf/onrobot_rg.urdf.xacro (robot description, xacro)
@@ -13,5 +13,5 @@
     <!-- load config from file -->
     <xacro:property name="config_file" value="$(find onrobot_description)/config/${model}.yaml"/>
-    <xacro:property name="config" value="${load_yaml(config_file)}"/>
+    <xacro:property name="config" value="${xacro.load_yaml(config_file)}"/>
     <xacro:property name="limit" value="${config['limit']}"/>
     <xacro:property name="origin" value="${config['origin']}"/>

Commit message: Replace xacro.load_yaml with load_yaml. Will create warnings in some cases but prevent crash for older xacro version (on conda)

File: onrobot_description/urdf/onrobot_rg.urdf.xacro (robot description, xacro)
@@ -13,5 +13,5 @@
     <!-- load config from file -->
     <xacro:property name="config_file" value="$(find onrobot_description)/config/${model}.yaml"/>
-    <xacro:property name="config" value="${xacro.load_yaml(config_file)}"/>
+    <xacro:property name="config" value="${load_yaml(config_file)}"/>
     <xacro:property name="limit" value="${config['limit']}"/>
     <xacro:property name="origin" value="${config['origin']}"/>
