Commit message: add gazebo sim

File: onrobot_description/urdf/onrobot_rg.gazebo.xacro (robot description, xacro)
@@ -1,7 +1,7 @@
 <?xml version="1.0"?>
 <robot xmlns:xacro="http://ros.org/wiki/xacro">
-  <xacro:macro name="rg_gazebo" params="prefix origin limit safety_shield:=False">
+  <xacro:macro name="rg_gazebo" params="prefix origin limit standalone:=True safety_shield:=False">
     <!-- load "onrobot_gripper_plugin" plugin -->
-    <gazebo>
+    <!-- <gazebo>
       <plugin name="${prefix}_plugin" filename="libonrobot_gripper_plugin.so">
         <robotNamespace>/${prefix}</robotNamespace>
@@ -14,5 +14,12 @@
         <maxEffort>0.5</maxEffort>
       </plugin>
-    </gazebo>
+    </gazebo> -->
+    <xacro:if value="${standalone}">
+      <gazebo>
+        <plugin filename="gz_ros2_control-system" name="gz_ros2_control::GazeboSimROS2ControlPlugin">
+            <parameters>$(find onrobot_control)/config/onrobot_rg_standalone.yaml</parameters>
+        </plugin>
+      </gazebo>
+    </xacro:if>
     <!-- add close loop joints -->
     <xacro:property name="x" value="${origin['moment_arm']['x']-origin['truss_arm']['x']}"/>
@@ -30,8 +37,8 @@
       </joint>
     </xacro:macro>
-    <gazebo>
+    <!-- <gazebo>
       <xacro:close_loop_joint name="${prefix}_finger_1"/>
       <xacro:close_loop_joint name="${prefix}_finger_2"/>
-    </gazebo>
+    </gazebo> -->
     <!-- tune tip's friction/collison model -->
     <xacro:macro name="grasp_friction" params="link_name">

File: onrobot_description/urdf/onrobot_rg.urdf.xacro (robot description, xacro)
@@ -9,6 +9,5 @@
   <!-- onrobot gripper -->
   <xacro:macro name="onrobot_rg" params="parent *origin prefix:='gripper'
-    model:='rg2_v1' safety_shield:=False bracket:='single_bracket' mount_angle:=0.0
-    transmission_hw_interface:=hardware_interface/EffortJointInterface">
+    model:='rg2_v1' safety_shield:=False bracket:='single_bracket' mount_angle:=0.0 standalone:=false real_hardware:=false">
     <!-- load config from file -->
     <xacro:property name="config_file" value="$(find onrobot_description)/config/${model}.yaml"/>
@@ -36,5 +35,5 @@
       <visual>
         <geometry>
-          <mesh filename="package://onrobot_description/meshes/${model}/visual/${bracket}.stl"/>
+          <mesh filename="file://$(find onrobot_description)/meshes/${model}/visual/${bracket}.stl"/>
         </geometry>
         <material name="onrobot/grey"/>
@@ -42,5 +41,5 @@
       <collision>
         <geometry>
-          <mesh filename="package://onrobot_description/meshes/${model}/collision/${bracket}.stl"/>
+          <mesh filename="file://$(find onrobot_description)/meshes/${model}/collision/${bracket}.stl"/>
         </geometry>
       </collision>
@@ -56,5 +55,5 @@
       <visual>
         <geometry>
-          <mesh filename="package://onrobot_description/meshes/${model}/visual/body.stl"/>
+          <mesh filename="file://$(find onrobot_description)/meshes/${model}/visual/body.stl"/>
         </geometry>
         <material name="onrobot/light_grey"/>
@@ -62,5 +61,5 @@
       <collision>
         <geometry>
-          <mesh filename="package://onrobot_description/meshes/${model}/collision/body.stl"/>
+          <mesh filename="file://$(find onrobot_description)/meshes/${model}/collision/body.stl"/>
         </geometry>
       </collision>
@@ -97,5 +96,5 @@
         <visual>
           <geometry>
-            <mesh filename="package://onrobot_description/meshes/${model}/visual/moment_arm.stl"/>
+            <mesh filename="file://$(find onrobot_description)/meshes/${model}/visual/moment_arm.stl"/>
           </geometry>
           <material name="onrobot/light_grey"/>
@@ -103,5 +102,5 @@
         <collision>
           <geometry>
-            <mesh filename="package://onrobot_description/meshes/${model}/collision/moment_arm.stl"/>
+            <mesh filename="file://$(find onrobot_description)/meshes/${model}/collision/moment_arm.stl"/>
           </geometry>
         </collision>
@@ -123,5 +122,5 @@
         <visual>
           <geometry>
-            <mesh filename="package://onrobot_description/meshes/${model}/visual/truss_arm.stl"/>
+            <mesh filename="file://$(find onrobot_description)/meshes/${model}/visual/truss_arm.stl"/>
           </geometry>
           <material name="onrobot/light_grey"/>
@@ -129,5 +128,5 @@
         <collision>
           <geometry>
-            <mesh filename="package://onrobot_description/meshes/${model}/collision/truss_arm.stl"/>
+            <mesh filename="file://$(find onrobot_description)/meshes/${model}/collision/truss_arm.stl"/>
           </geometry>
         </collision>
@@ -147,5 +146,5 @@
           <visual>
             <geometry>
-              <mesh filename="package://onrobot_description/meshes/${model}/visual/safety_shield.stl"/>
+              <mesh filename="file://$(find onrobot_description)/meshes/${model}/visual/safety_shield.stl"/>
             </geometry>
             <material name="onrobot/dark_grey"/>
@@ -153,5 +152,5 @@
           <collision>
             <geometry>
-              <!-- <mesh filename="package://onrobot_description/meshes/${model}/collision/safety_shield.stl"/> -->
+              <mesh filename="file://$(find onrobot_description)/meshes/${model}/collision/safety_shield.stl"/>
               <box size="0.0 0.0 0.0"/>
             </geometry>
@@ -172,5 +171,5 @@
         <visual>
           <geometry>
-            <mesh filename="package://onrobot_description/meshes/${model}/visual/finger_tip.stl"/>
+            <mesh filename="file://$(find onrobot_description)/meshes/${model}/visual/finger_tip.stl"/>
           </geometry>
           <material name="onrobot/light_grey"/>
@@ -178,10 +177,10 @@
         <collision>
           <geometry>
-            <mesh filename="package://onrobot_description/meshes/${model}/collision/finger_tip_1.stl"/>
-          </geometry>
-        </collision>
-        <collision>
-          <geometry>
-            <mesh filename="package://onrobot_description/meshes/${model}/collision/finger_tip_2.stl"/>
+            <mesh filename="file://$(find onrobot_description)/meshes/${model}/collision/finger_tip_1.stl"/>
+          </geometry>
+        </collision>
+        <collision>
+          <geometry>
+            <mesh filename="file://$(find onrobot_description)/meshes/${model}/collision/finger_tip_2.stl"/>
           </geometry>
         </collision>
@@ -200,5 +199,5 @@
         <visual>
           <geometry>
-            <mesh filename="package://onrobot_description/meshes/${model}/visual/flex_finger.stl"/>
+            <mesh filename="file://$(find onrobot_description)/meshes/${model}/visual/flex_finger.stl"/>
           </geometry>
           <material name="onrobot/dark_grey"/>
@@ -206,5 +205,5 @@
         <collision>
           <geometry>
-            <mesh filename="package://onrobot_description/meshes/${model}/collision/flex_finger.stl"/>
+            <mesh filename="file://$(find onrobot_description)/meshes/${model}/collision/flex_finger.stl"/>
           </geometry>
         </collision>
@@ -219,6 +218,41 @@
     <xacro:finger name="${prefix}_finger_1" is_master="true"/>
     <xacro:finger name="${prefix}_finger_2" is_master="false"/>
-    <xacro:rg_transmission prefix="${prefix}" hw_interface="${transmission_hw_interface}"/>
-    <xacro:rg_gazebo prefix="${prefix}" origin="${origin}" limit="${limit}" safety_shield="${safety_shield}"/>
+    <ros2_control name="${prefix}" type="system">
+          <hardware>
+              <plugin>gz_ros2_control/GazeboSimSystem</plugin>
+          </hardware>
+          <joint name="${prefix}_joint">
+              <command_interface name="position"/>
+              <state_interface name="position">
+                    <!-- <param name="initial_value">1.</param> -->
+              </state_interface>
+              <state_interface name="velocity"/>
+              <state_interface name="effort"/>
+          </joint>
+          <joint name="${prefix}_finger_1_truss_arm_joint">
+            <state_interface name="position"/>
+          </joint>
+          <joint name="${prefix}_finger_1_finger_tip_joint">
+            <state_interface name="position"/>
+          </joint>
+          <xacro:if value="${safety_shield}">
+            <joint name="${prefix}_finger_1_safety_shield_joint">
+              <state_interface name="position"/>
+            </joint>
+          </xacro:if>
+          <joint name="${prefix}_finger_2_truss_arm_joint">
+            <state_interface name="position"/>
+          </joint>
+          <joint name="${prefix}_finger_2_finger_tip_joint">
+            <state_interface name="position"/>
+          </joint>
+          <xacro:if value="${safety_shield}">
+            <joint name="${prefix}_finger_2_safety_shield_joint">
+              <state_interface name="position"/>
+            </joint>
+          </xacro:if>
+    </ros2_control>
+    <!-- si standalone alors mettre le plugin de ros2_control -->
+    <xacro:rg_gazebo prefix="${prefix}" origin="${origin}" limit="${limit}" standalone="${standalone}" safety_shield="${safety_shield}"/>
   </xacro:macro>
 </robot>

File: onrobot_description/urdf/test.urdf.xacro (robot description, xacro)
@@ -3,9 +3,20 @@
   <xacro:include filename="$(find onrobot_description)/urdf/onrobot_rg.urdf.xacro" />
   <link name="world" />
-  <xacro:onrobot_rg parent="world" model='rg2_v1' prefix='rg2'>
-    <origin xyz="0.0 0.05 0.0" rpy="0.0 0.0 0.0" />
-  </xacro:onrobot_rg>
-  <xacro:onrobot_rg parent="world" model='rg6_v1' safety_shield='true' prefix='rg6'>
-    <origin xyz="0.0 -0.05 0.0" rpy="0.0 0.0 0.0" />
-  </xacro:onrobot_rg>
+  <xacro:arg name="model" default="rg2_v1" />
+  <xacro:property name="model_prop" value="$(arg model)" />
+  <xacro:if value="${model_prop == 'rg2_v1'}">
+    <xacro:onrobot_rg parent="world" model='rg2_v1' prefix='rg2' standalone='true'>
+      <origin xyz="0.0 0.05 0.01" rpy="0.0 0.0 0.0" />
+    </xacro:onrobot_rg>
+  </xacro:if>
+  <xacro:if value="${model_prop == 'rg6_v1'}">
+    <xacro:onrobot_rg parent="world" model='rg6_v1' prefix='rg6' standalone='true'>
+      <origin xyz="0.0 0.05 0.01" rpy="0.0 0.0 0.0" />
+    </xacro:onrobot_rg>
+  </xacro:if>
+  <xacro:if value="${model_prop == 'rg6_v2'}">
+    <xacro:onrobot_rg parent="world" model='rg6_v2' prefix='rg6' standalone='true'>
+      <origin xyz="0.0 0.05 0.01" rpy="0.0 0.0 0.0" />
+    </xacro:onrobot_rg>
+  </xacro:if>
 </robot>

Commit message: hardware interface add

File: onrobot_description/urdf/onrobot_rg.gazebo.xacro (robot description, xacro)
@@ -62,6 +62,6 @@
       </gazebo>
     </xacro:macro>
-    <xacro:grasp_friction link_name="${prefix}_finger_1_flex_finger"/>
-    <xacro:grasp_friction link_name="${prefix}_finger_2_flex_finger"/>
+    <!-- <xacro:grasp_friction link_name="${prefix}_finger_1_flex_finger"/> -->
+    <!-- <xacro:grasp_friction link_name="${prefix}_finger_2_flex_finger"/> -->
     <!-- enable self collision -->
     <gazebo reference="${prefix}_bracket">

File: onrobot_description/urdf/onrobot_rg.urdf.xacro (robot description, xacro)
@@ -8,6 +8,7 @@
   <xacro:include filename="$(find onrobot_description)/urdf/onrobot_rg.gazebo.xacro" />
   <!-- onrobot gripper -->
-  <xacro:macro name="onrobot_rg" params="parent *origin prefix:='gripper'
+  <xacro:macro name="onrobot_rg" params="parent *origin prefix:=''
     model:='rg2_v1' safety_shield:=False bracket:='single_bracket' mount_angle:=0.0 standalone:=false real_hardware:=false">
+    <xacro:property name="gripper_name" value="${prefix}gripper"/>
     <!-- load config from file -->
     <xacro:property name="config_file" value="$(find onrobot_description)/config/${model}.yaml"/>
@@ -32,5 +33,5 @@
     </xacro:macro>
     <!-- bracket -->
-    <link name="${prefix}_bracket">
+    <link name="${gripper_name}_bracket">
       <visual>
         <geometry>
@@ -46,11 +47,11 @@
       <xacro:_inertial id="${bracket}"/>
     </link>
-    <joint name="${prefix}_bracket_joint" type="fixed">
+    <joint name="${gripper_name}_bracket_joint" type="fixed">
       <parent link="${parent}"/>
-      <child link = "${prefix}_bracket"/>
+      <child link = "${gripper_name}_bracket"/>
       <xacro:insert_block name="origin"/>
     </joint>
     <!-- body -->
-    <link name="${prefix}_body">
+    <link name="${gripper_name}_body">
       <visual>
         <geometry>
@@ -66,14 +67,14 @@
       <xacro:_inertial id="body"/>
     </link>
-    <joint name="${prefix}_body_joint" type="fixed">
-      <parent link="${prefix}_bracket"/>
-      <child link = "${prefix}_body"/>
+    <joint name="${gripper_name}_body_joint" type="fixed">
+      <parent link="${gripper_name}_bracket"/>
+      <child link = "${gripper_name}_body"/>
       <xacro:_frame id="${bracket}" rpy="${mount_angle} 0.0 0.0"/>
     </joint>
     <!-- grasp frame -->
-    <link name="${prefix}_grasp_frame"/>
-    <joint name="${prefix}_grasp_frame_joint" type="fixed">
-      <parent link="${prefix}_body"/>
-      <child link = "${prefix}_grasp_frame"/>
+    <link name="${gripper_name}_grasp_frame"/>
+    <joint name="${gripper_name}_grasp_frame_joint" type="fixed">
+      <parent link="${gripper_name}_body"/>
+      <child link = "${gripper_name}_grasp_frame"/>
       <xacro:_frame id="grasp_frame" rpy="0.0 0.0 0.0"/>
     </joint>
@@ -88,5 +89,5 @@
       </link>
       <joint name="${name}_origin_joint" type="fixed">
-        <parent link="${prefix}_body"/>
+        <parent link="${gripper_name}_body"/>
         <child link = "${name}_origin"/>
         <origin xyz="0 0 0" rpy="0 0 ${0 if is_master else pi}"/>
@@ -107,5 +108,5 @@
         <xacro:_inertial id="moment_arm"/>
       </link>
-      <joint name="${prefix + ('' if is_master else '_mirror')}_joint" type="revolute">
+      <joint name="${gripper_name + ('' if is_master else '_mirror')}_joint" type="revolute">
         <parent link="${name}_origin"/>
         <child link = "${name}_moment_arm"/>
@@ -113,7 +114,7 @@
         <xacro:_frame id="moment_arm" rpy="0.0 ${offset} 0.0"/>
         <xacro:_limit/>
-        <dynamics damping="0.5"/>
+        <!-- <dynamics damping="0.5"/> -->
         <xacro:unless value="${is_master}">
-          <mimic joint="${prefix}_joint" multiplier="1" offset="0"/>
+          <mimic joint="${gripper_name}_joint" multiplier="1" offset="0"/>
         </xacro:unless>
       </joint>
@@ -139,5 +140,5 @@
         <xacro:_frame id="truss_arm" rpy="0.0 ${offset} 0.0"/>
         <xacro:_limit/>
-        <mimic joint="${prefix}_joint" multiplier="1" offset="0"/>
+        <mimic joint="${gripper_name}_joint" multiplier="1" offset="0"/>
       </joint>
       <!-- safety shield -->
@@ -164,5 +165,5 @@
           <xacro:_frame id="safety_shield" rpy="0.0 ${offset} 0.0"/>
           <xacro:_limit/>
-          <mimic joint="${prefix}_joint" multiplier="1" offset="0"/>
+          <mimic joint="${gripper_name}_joint" multiplier="1" offset="0"/>
         </joint>
       </xacro:if>
@@ -193,5 +194,5 @@
         <xacro:_frame id="finger_tip" rpy="0.0 ${-offset} 0.0"/>
         <xacro:_limit/>
-        <mimic joint="${prefix}_joint" multiplier="1" offset="0"/>
+        <mimic joint="${gripper_name}_joint" multiplier="1" offset="0"/>
       </joint>
       <!-- flex finger -->
@@ -216,43 +217,59 @@
       </joint>
     </xacro:macro>
-    <xacro:finger name="${prefix}_finger_1" is_master="true"/>
-    <xacro:finger name="${prefix}_finger_2" is_master="false"/>
-    <ros2_control name="${prefix}" type="system">
-          <hardware>
-              <plugin>gz_ros2_control/GazeboSimSystem</plugin>
-          </hardware>
-          <joint name="${prefix}_joint">
-              <command_interface name="position"/>
-              <state_interface name="position">
-                    <!-- <param name="initial_value">1.</param> -->
-              </state_interface>
-              <state_interface name="velocity"/>
-              <state_interface name="effort"/>
-          </joint>
-          <joint name="${prefix}_finger_1_truss_arm_joint">
-            <state_interface name="position"/>
-          </joint>
-          <joint name="${prefix}_finger_1_finger_tip_joint">
-            <state_interface name="position"/>
-          </joint>
-          <xacro:if value="${safety_shield}">
-            <joint name="${prefix}_finger_1_safety_shield_joint">
-              <state_interface name="position"/>
-            </joint>
-          </xacro:if>
-          <joint name="${prefix}_finger_2_truss_arm_joint">
-            <state_interface name="position"/>
-          </joint>
-          <joint name="${prefix}_finger_2_finger_tip_joint">
-            <state_interface name="position"/>
-          </joint>
-          <xacro:if value="${safety_shield}">
-            <joint name="${prefix}_finger_2_safety_shield_joint">
-              <state_interface name="position"/>
+    <xacro:finger name="${gripper_name}_finger_1" is_master="true"/>
+    <xacro:finger name="${gripper_name}_finger_2" is_master="false"/>
+    <ros2_control name="${gripper_name}" type="system" is_async="true">
+          <xacro:unless value="${real_hardware}">
+            <hardware>
+                <plugin>gz_ros2_control/GazeboSimSystem</plugin>
+            </hardware>
+            <joint name="${gripper_name}_joint">
+                <command_interface name="position"/>
+                <state_interface name="position">
+                      <param name="initial_value">0.01</param> # avoid to be stuck due to a pos under 0.0
+                </state_interface>
+                <state_interface name="velocity"/>
+                <state_interface name="effort"/>
+            </joint>
+            <joint name="${gripper_name}_finger_1_truss_arm_joint">
+              <state_interface name="position"/>
+            </joint>
+            <joint name="${gripper_name}_finger_1_finger_tip_joint">
+              <state_interface name="position"/>
+            </joint>
+            <xacro:if value="${safety_shield}">
+              <joint name="${gripper_name}_finger_1_safety_shield_joint">
+                <state_interface name="position"/>
+              </joint>
+            </xacro:if>
+            <joint name="${gripper_name}_finger_2_truss_arm_joint">
+              <state_interface name="position"/>
+            </joint>
+            <joint name="${gripper_name}_finger_2_finger_tip_joint">
+              <state_interface name="position"/>
+            </joint>
+            <xacro:if value="${safety_shield}">
+              <joint name="${gripper_name}_finger_2_safety_shield_joint">
+                <state_interface name="position"/>
+              </joint>
+            </xacro:if>
+          </xacro:unless>
+          <xacro:if value="${real_hardware}">
+            <hardware>
+                <plugin>onrobot_interface::OnRobotHardwareInterface</plugin>
+                <param name="prefix">${prefix}</param>
+            </hardware>
+            <joint name="${gripper_name}_joint">
+                <command_interface name="position"/>
+                <state_interface name="position"/>
+                <state_interface name="velocity"/>
+                <state_interface name="effort"/>
             </joint>
           </xacro:if>
     </ros2_control>
     <!-- si standalone alors mettre le plugin de ros2_control -->
-    <xacro:rg_gazebo prefix="${prefix}" origin="${origin}" limit="${limit}" standalone="${standalone}" safety_shield="${safety_shield}"/>
+    <xacro:unless value="${real_hardware}">
+      <xacro:rg_gazebo prefix="${gripper_name}" origin="${origin}" limit="${limit}" standalone="${standalone}" safety_shield="${safety_shield}"/>
+    </xacro:unless>
   </xacro:macro>
 </robot>

File: onrobot_description/urdf/test.urdf.xacro (robot description, xacro)
@@ -7,5 +7,5 @@
   <xacro:if value="${model_prop == 'rg2_v1'}">
     <xacro:onrobot_rg parent="world" model='rg2_v1' prefix='rg2' standalone='true'>
-      <origin xyz="0.0 0.05 0.01" rpy="0.0 0.0 0.0" />
+      <origin xyz="0.0 0.05 0.01" rpy="3.14 0.0 0.0" />
     </xacro:onrobot_rg>
   </xacro:if>
