Commit message: update voltage pos

File: onrobot_description/urdf/onrobot_rg.gazebo.xacro (robot description, xacro)
@@ -62,6 +62,6 @@
       </gazebo>
     </xacro:macro>
-    <!-- <xacro:grasp_friction link_name="${prefix}_finger_1_flex_finger"/> -->
-    <!-- <xacro:grasp_friction link_name="${prefix}_finger_2_flex_finger"/> -->
+    <xacro:grasp_friction link_name="${prefix}_finger_1_flex_finger"/>
+    <xacro:grasp_friction link_name="${prefix}_finger_2_flex_finger"/>
     <!-- enable self collision -->
     <gazebo reference="${prefix}_bracket">

File: onrobot_description/urdf/onrobot_rg.urdf.xacro (robot description, xacro)
@@ -42,5 +42,5 @@
       <collision>
         <geometry>
-          <mesh filename="file://$(find onrobot_description)/meshes/${model}/collision/${bracket}.stl"/>
+          <mesh filename="file://$(find onrobot_description)/meshes/${model}/visual/${bracket}.stl"/>
         </geometry>
       </collision>
@@ -62,5 +62,5 @@
       <collision>
         <geometry>
-          <mesh filename="file://$(find onrobot_description)/meshes/${model}/collision/body.stl"/>
+          <mesh filename="file://$(find onrobot_description)/meshes/${model}/visual/body.stl"/>
         </geometry>
       </collision>
@@ -103,5 +103,5 @@
         <collision>
           <geometry>
-            <mesh filename="file://$(find onrobot_description)/meshes/${model}/collision/moment_arm.stl"/>
+            <mesh filename="file://$(find onrobot_description)/meshes/${model}/visual/moment_arm.stl"/>
           </geometry>
         </collision>
@@ -114,5 +114,5 @@
         <xacro:_frame id="moment_arm" rpy="0.0 ${offset} 0.0"/>
         <xacro:_limit/>
-        <!-- <dynamics damping="0.5"/> -->
+        <dynamics damping="0.17"/>
         <xacro:unless value="${is_master}">
           <mimic joint="${gripper_name}_joint" multiplier="1" offset="0"/>
@@ -129,5 +129,5 @@
         <collision>
           <geometry>
-            <mesh filename="file://$(find onrobot_description)/meshes/${model}/collision/truss_arm.stl"/>
+            <mesh filename="file://$(find onrobot_description)/meshes/${model}/visual/truss_arm.stl"/>
           </geometry>
         </collision>
@@ -153,5 +153,5 @@
           <collision>
             <geometry>
-              <mesh filename="file://$(find onrobot_description)/meshes/${model}/collision/safety_shield.stl"/>
+              <mesh filename="file://$(find onrobot_description)/meshes/${model}/visual/safety_shield.stl"/>
               <box size="0.0 0.0 0.0"/>
             </geometry>
@@ -178,10 +178,10 @@
         <collision>
           <geometry>
-            <mesh filename="file://$(find onrobot_description)/meshes/${model}/collision/finger_tip_1.stl"/>
-          </geometry>
-        </collision>
-        <collision>
-          <geometry>
-            <mesh filename="file://$(find onrobot_description)/meshes/${model}/collision/finger_tip_2.stl"/>
+            <mesh filename="file://$(find onrobot_description)/meshes/${model}/visual/finger_tip.stl"/>
+          </geometry>
+        </collision>
+        <collision>
+          <geometry>
+            <mesh filename="file://$(find onrobot_description)/meshes/${model}/visual/finger_tip.stl"/>
           </geometry>
         </collision>
@@ -206,5 +206,5 @@
         <collision>
           <geometry>
-            <mesh filename="file://$(find onrobot_description)/meshes/${model}/collision/flex_finger.stl"/>
+            <mesh filename="file://$(find onrobot_description)/meshes/${model}/visual/flex_finger.stl"/>
           </geometry>
         </collision>

File: onrobot_description/urdf/test.urdf.xacro (robot description, xacro)
@@ -6,15 +6,15 @@
   <xacro:property name="model_prop" value="$(arg model)" />
   <xacro:if value="${model_prop == 'rg2_v1'}">
-    <xacro:onrobot_rg parent="world" model='rg2_v1' prefix='rg2' standalone='true'>
-      <origin xyz="0.0 0.05 0.01" rpy="3.14 0.0 0.0" />
+    <xacro:onrobot_rg parent="world" model='rg2_v1' prefix='rg2_' standalone='true' real_hardware='false'>
+      <origin xyz="2. 0.05 2." rpy="1.5708 -1.5708 0.0" />
     </xacro:onrobot_rg>
   </xacro:if>
   <xacro:if value="${model_prop == 'rg6_v1'}">
-    <xacro:onrobot_rg parent="world" model='rg6_v1' prefix='rg6' standalone='true'>
+    <xacro:onrobot_rg parent="world" model='rg6' prefix='rg6_' standalone='true' real_hardware='false'>
       <origin xyz="0.0 0.05 0.01" rpy="0.0 0.0 0.0" />
     </xacro:onrobot_rg>
   </xacro:if>
   <xacro:if value="${model_prop == 'rg6_v2'}">
-    <xacro:onrobot_rg parent="world" model='rg6_v2' prefix='rg6' standalone='true'>
+    <xacro:onrobot_rg parent="world" model='rg6_v2' prefix='rg6_v2_' standalone='true' real_hardware='false'>
       <origin xyz="0.0 0.05 0.01" rpy="0.0 0.0 0.0" />
     </xacro:onrobot_rg>

Commit message: closed loop  test

File: onrobot_description/urdf/onrobot_rg.gazebo.xacro (robot description, xacro)
@@ -62,8 +62,8 @@
       </gazebo>
     </xacro:macro>
-    <xacro:grasp_friction link_name="${prefix}_finger_1_flex_finger"/>
-    <xacro:grasp_friction link_name="${prefix}_finger_2_flex_finger"/>
+    <!-- <xacro:grasp_friction link_name="${prefix}_finger_1_flex_finger"/> -->
+    <!-- <xacro:grasp_friction link_name="${prefix}_finger_2_flex_finger"/> -->
     <!-- enable self collision -->
-    <gazebo reference="${prefix}_bracket">
+    <!-- <gazebo reference="${prefix}_bracket">
       <selfCollide>true</selfCollide>
     </gazebo>
@@ -94,5 +94,5 @@
     <gazebo reference="${prefix}_finger_2_flex_finger">
       <selfCollide>true</selfCollide>
-    </gazebo>
+    </gazebo> -->
   </xacro:macro>
 </robot>

File: onrobot_description/urdf/onrobot_rg.urdf.xacro (robot description, xacro)
@@ -112,5 +112,5 @@
         <child link = "${name}_moment_arm"/>
         <axis xyz="0 1 0"/>
-        <xacro:_frame id="moment_arm" rpy="0.0 ${offset} 0.0"/>
+        <xacro:_frame id="moment_arm" rpy="0.0 ${offset-0.01} 0.0"/>
         <xacro:_limit/>
         <dynamics damping="0.17"/>
@@ -140,5 +140,4 @@
         <xacro:_frame id="truss_arm" rpy="0.0 ${offset} 0.0"/>
         <xacro:_limit/>
-        <mimic joint="${gripper_name}_joint" multiplier="1" offset="0"/>
       </joint>
       <!-- safety shield -->
@@ -165,5 +164,4 @@
           <xacro:_frame id="safety_shield" rpy="0.0 ${offset} 0.0"/>
           <xacro:_limit/>
-          <mimic joint="${gripper_name}_joint" multiplier="1" offset="0"/>
         </joint>
       </xacro:if>
@@ -194,5 +192,4 @@
         <xacro:_frame id="finger_tip" rpy="0.0 ${-offset} 0.0"/>
         <xacro:_limit/>
-        <mimic joint="${gripper_name}_joint" multiplier="1" offset="0"/>
       </joint>
       <!-- flex finger -->
@@ -215,4 +212,18 @@
         <child link = "${name}_flex_finger"/>
         <xacro:_frame id="flex_finger" rpy="0.0 0.0 0.0"/>
+      </joint>
+      <!-- dummy link for detach/attach object in gazebo -->
+      <link name="${name}_dummy_link">
+        <inertial>
+          <mass value="0.001"/>
+          <inertia ixx="0.00001" ixy="0.0" ixz="0.0" iyy="0.00001" iyz="0.0" izz="0.00001"/>
+        </inertial>
+      </link>
+      <joint name="${name}_dummy_link_joint" type="revolute">
+        <parent link="${name}_moment_arm"/>
+        <child link = "${name}_dummy_link"/>
+        <axis xyz="0 1 0"/>
+        <origin xyz="${origin['finger_tip']['x']} ${origin['finger_tip']['y']} ${origin['finger_tip']['z']}" rpy="0.0 ${offset} 0.0"/>
+        <xacro:_limit/>
       </joint>
     </xacro:macro>
@@ -232,4 +243,9 @@
                 <state_interface name="effort"/>
             </joint>
+            <joint name="${gripper_name}_mirror_joint">
+              <state_interface name="position"/>
+              <state_interface name="velocity"/>
+              <state_interface name="effort"/>
+            </joint>
             <joint name="${gripper_name}_finger_1_truss_arm_joint">
               <state_interface name="position"/>
@@ -254,4 +270,10 @@
               </joint>
             </xacro:if>
+            <joint name="${gripper_name}_finger_1_dummy_link_joint">
+              <state_interface name="position"/>
+            </joint>
+            <joint name="${gripper_name}_finger_2_dummy_link_joint">
+              <state_interface name="position"/>
+            </joint>
           </xacro:unless>
           <xacro:if value="${real_hardware}">
@@ -269,8 +291,81 @@
           </xacro:if>
     </ros2_control>
+    <gazebo>
+      <!-- Connect moment arm to finger tip (via dummy_link) -->
+      <plugin filename="libgz-sim-detachable-joint-system.so" name="gz::sim::systems::DetachableJoint">
+          <parent_link>${gripper_name}_finger_1_finger_tip</parent_link>
+          <child_model>${model}</child_model>
+          <child_link>${gripper_name}_finger_1_dummy_link</child_link>
+          <attach_topic>loop/attach</attach_topic>
+          <detach_topic>loop/detach</detach_topic>
+          <output_topic>loop/state</output_topic>
+      </plugin>
+      <plugin filename="libgz-sim-detachable-joint-system.so" name="gz::sim::systems::DetachableJoint">
+          <parent_link>${gripper_name}_finger_2_finger_tip</parent_link>
+          <child_model>${model}</child_model>
+          <child_link>${gripper_name}_finger_2_dummy_link</child_link>
+          <attach_topic>loop/attach</attach_topic>
+          <detach_topic>loop/detach</detach_topic>
+          <output_topic>loop/state</output_topic>
+      </plugin>
+    </gazebo>
     <!-- si standalone alors mettre le plugin de ros2_control -->
     <xacro:unless value="${real_hardware}">
       <xacro:rg_gazebo prefix="${gripper_name}" origin="${origin}" limit="${limit}" standalone="${standalone}" safety_shield="${safety_shield}"/>
     </xacro:unless>
+     <gazebo reference="${prefix}gripper_bracket">
+    <selfCollide>false</selfCollide>
+    </gazebo>
+    <gazebo reference="${prefix}gripper_body">
+      <selfCollide>false</selfCollide>
+    </gazebo>
+    <!-- Doigt 1 -->
+    <gazebo reference="${prefix}gripper_finger_1_origin">
+      <selfCollide>false</selfCollide>
+    </gazebo>
+    <gazebo reference="${prefix}gripper_finger_1_moment_arm">
+      <selfCollide>false</selfCollide>
+    </gazebo>
+    <gazebo reference="${prefix}gripper_finger_1_truss_arm">
+      <selfCollide>false</selfCollide>
+    </gazebo>
+    <gazebo reference="${prefix}gripper_finger_1_finger_tip">
+      <selfCollide>false</selfCollide>
+    </gazebo>
+    <gazebo reference="${prefix}gripper_finger_1_flex_finger">
+      <selfCollide>false</selfCollide>
+    </gazebo>
+    <gazebo reference="${prefix}gripper_finger_1_dummy_link">
+      <selfCollide>false</selfCollide>
+    </gazebo>
+    <xacro:if value="${safety_shield}">
+      <gazebo reference="${prefix}gripper_finger_1_safety_shield">
+          <selfCollide>false</selfCollide>
+      </gazebo>
+    </xacro:if>
+    <!-- Doigt 2 -->
+    <gazebo reference="${prefix}gripper_finger_2_origin">
+      <selfCollide>false</selfCollide>
+    </gazebo>
+    <gazebo reference="${prefix}gripper_finger_2_moment_arm">
+      <selfCollide>false</selfCollide>
+    </gazebo>
+    <gazebo reference="${prefix}gripper_finger_2_truss_arm">
+      <selfCollide>false</selfCollide>
+    </gazebo>
+    <gazebo reference="${prefix}gripper_finger_2_finger_tip">
+      <selfCollide>false</selfCollide>
+    </gazebo>
+    <gazebo reference="${prefix}gripper_finger_2_flex_finger">
+      <selfCollide>false</selfCollide>
+    </gazebo>
+    <gazebo reference="${prefix}gripper_finger_2_dummy_link">
+      <selfCollide>false</selfCollide>
+    </gazebo>
+    <xacro:if value="${safety_shield}">
+      <gazebo reference="${prefix}gripper_finger_2_safety_shield">
+          <selfCollide>false</selfCollide>
+      </gazebo>
+    </xacro:if>
   </xacro:macro>
 </robot>

File: onrobot_description/urdf/test.urdf.xacro (robot description, xacro)
@@ -1,5 +1,6 @@
 <?xml version="1.0"?>
-<robot xmlns:xacro="http://wiki.ros.org/xacro" name="onrobot_rg_test">
-  <xacro:include filename="$(find onrobot_description)/urdf/onrobot_rg.urdf.xacro" />
+<robot xmlns:xacro="http://www.ros.org/xacro" name="rg2_standalone">
+    <!-- 1. Inclure la macro de votre gripper -->
+    <xacro:include filename="$(find onrobot_description)/urdf/onrobot_rg.urdf.xacro" />
   <link name="world" />
   <xacro:arg name="model" default="rg2_v1" />
@@ -7,9 +8,9 @@
   <xacro:if value="${model_prop == 'rg2_v1'}">
     <xacro:onrobot_rg parent="world" model='rg2_v1' prefix='rg2_' standalone='true' real_hardware='false'>
-      <origin xyz="2. 0.05 2." rpy="1.5708 -1.5708 0.0" />
+      <origin xyz="0.0 0.05 0.01" rpy="0.0 0.0 0.0" />
     </xacro:onrobot_rg>
   </xacro:if>
   <xacro:if value="${model_prop == 'rg6_v1'}">
-    <xacro:onrobot_rg parent="world" model='rg6' prefix='rg6_' standalone='true' real_hardware='false'>
+    <xacro:onrobot_rg parent="world" model='rg6_v1' prefix='rg6_' standalone='true' real_hardware='false'>
       <origin xyz="0.0 0.05 0.01" rpy="0.0 0.0 0.0" />
     </xacro:onrobot_rg>
